Commit message: Thorvald full URDF

File: urdf/macros.xacro (robot description, xacro)
@@ -8,5 +8,5 @@
             <visual>
                 <geometry>
-                    <mesh filename="package://oxar_is_bored/mesh/${filename}" scale="0.001 0.001 0.001"/>
+                    <mesh filename="package://oxar_is_bored/meshes/${filename}" scale="0.001 0.001 0.001"/>
                 </geometry>
                 <xacro:white_material/>
