Commit message: Animated arms on thorvald

File: urdf/arm.xacro (robot description, xacro)
@@ -11,5 +11,5 @@
             <origin xyz="${xyz}" rpy="${rpy}"/>
             <axis xyz="0 0 1"/>
-            <limit effort="10" lower="0" upper="0.5" velocity="0.5"/>
+            <limit effort="10" lower="-0.5" upper="0" velocity="0.5"/>
         </joint>
         <!-- Joint 1 -->

File: urdf/thorvald_full.xacro (robot description, xacro)
@@ -4,5 +4,10 @@
     <xacro:include filename="thorvald_base.urdf.xacro"/>
     <xacro:include filename="thorvald_arc.urdf.xacro"/>
-    <!-- Create arc -->
-    <xacro:thorvald_arc xyz="-0.5 0 0.5"/>
+    <xacro:include filename="arm.xacro"/>
+    <!-- Arc -->
+    <xacro:thorvald_arc name="arc_link" xyz="-0.5 0 0.5"/>
+    <!-- Arm1 -->
+    <xacro:thorvald_arm name="armL" parent="arc_link" xyz="0.55 -0.55 0.2" rpy="0 0 0"/>
+    <!-- Arm2 -->
+    <xacro:thorvald_arm name="armR" parent="arc_link" xyz="0.55 0.55 0.2" rpy="0 0 3.14"/>
 </robot>

Commit message: Add markers to end effector

File: urdf/arm.xacro (robot description, xacro)
@@ -58,4 +58,10 @@
             <limit effort="10.0" velocity="1.0" lower="-2" upper="2"/>
         </joint>
+        <link name="${name}_end_effector_link"/>
+        <joint name="${name}_joint_6" type="fixed">
+            <parent link="${name}_end2_link"/>
+            <child link="${name}_end_effector_link"/>
+            <origin xyz="0.04 -0.016 0" rpy="0 0 0"/>
+        </joint>
     </xacro:macro>
 </robot>

Commit message: Add markers to end effector

File: urdf/arm.xacro (robot description, xacro)
@@ -67,5 +67,9 @@
         <link name="${name}_end_effector_link"/>
         <joint name="${name}_joint_6" type="fixed">
+<<<<<<< HEAD
             <parent link="${name}_tilt_link"/>
+=======
+            <parent link="${name}_end2_link"/>
+>>>>>>> 0a74866... Add markers to end effector
             <child link="${name}_end_effector_link"/>
             <origin xyz="0.04 -0.016 0" rpy="0 0 0"/>

Commit message: Target reference

File: urdf/arm.xacro (robot description, xacro)
@@ -6,16 +6,23 @@
         <!-- Base Link -->
         <link name="${name}_base_link"/>
-        <joint name="${name}_base_joint" type="prismatic">
+        <joint name="${name}_base_joint" type="fixed">
+            <origin xyz="${xyz}" rpy="${rpy}"/>
             <parent link="${parent}"/>
             <child link="${name}_base_link"/>
-            <origin xyz="${xyz}" rpy="${rpy}"/>
+        </joint>
+        <!-- Prismatic Link -->
+        <link name="${name}_prismatic_link"/>
+        <joint name="${name}_prismatic_joint" type="prismatic">
+            <parent link="${name}_base_link"/>
+            <child link="${name}_prismatic_link"/>
+            <origin xyz="0 0 0" rpy="0 0 0"/>
             <axis xyz="0 0 1"/>
             <limit effort="10" lower="-0.5" upper="0" velocity="0.5"/>
         </joint>
         <!-- Joint 1 -->
-        <xacro:stl name="${name}_arm1_link" filename="Arm_joint_1.stl"/>
+        <xacro:stl name="${name}_shoulder_link" filename="Arm_joint_1.stl"/>
         <joint name="${name}_joint_1" type="revolute">
-            <parent link="${name}_base_link"/>
-            <child link="${name}_arm1_link"/>
+            <parent link="${name}_prismatic_link"/>
+            <child link="${name}_shoulder_link"/>
             <origin xyz="0 0 0" rpy="0 0 0"/>
             <axis xyz="0 0 1"/>
@@ -23,8 +30,8 @@
         </joint>
         <!-- Joint 2 -->
-        <xacro:stl name="${name}_arm2_link" filename="Arm_joint_2.stl"/>
+        <xacro:stl name="${name}_forearm_link" filename="Arm_joint_2.stl"/>
         <joint name="${name}_joint_2" type="revolute">
-            <parent link="${name}_arm1_link"/>
-            <child link="${name}_arm2_link"/>
+            <parent link="${name}_shoulder_link"/>
+            <child link="${name}_forearm_link"/>
             <origin xyz="0 0.2 0" rpy="0 0 0"/>
             <axis xyz="0 0 1"/>
@@ -32,8 +39,8 @@
         </joint>
         <!-- Joint 3 -->
-        <xacro:stl name="${name}_base_offset_link" filename="End effector.stl"/>
+        <xacro:stl name="${name}_offset_link" filename="End effector.stl"/>
         <joint name="${name}_joint_3" type="revolute">
-            <parent link="${name}_arm2_link"/>
-            <child link="${name}_base_offset_link"/>
+            <parent link="${name}_forearm_link"/>
+            <child link="${name}_offset_link"/>
             <origin xyz="0 0.16 0.025" rpy="1.57 0 0"/>
             <axis xyz="0 1 0"/>
@@ -41,8 +48,8 @@
         </joint>
         <!-- Joint 4 -->
-        <xacro:stl name="${name}_end1_link" filename="End_joint_1.stl"/>
+        <xacro:stl name="${name}_pan_link" filename="End_joint_1.stl"/>
         <joint name="${name}_joint_4" type="revolute">
-            <parent link="${name}_base_offset_link"/>
-            <child link="${name}_end1_link"/>
+            <parent link="${name}_offset_link"/>
+            <child link="${name}_pan_link"/>
             <origin xyz="0 0.223 -0.02" rpy="0 1.57 0"/>
             <axis xyz="0 1 0"/>
@@ -50,8 +57,8 @@
         </joint>
         <!-- Joint 5 -->
-        <xacro:stl name="${name}_end2_link" filename="End_joint_2.stl"/>
+        <xacro:stl name="${name}_tilt_link" filename="End_joint_2.stl"/>
         <joint name="${name}_joint_5" type="revolute">
-            <parent link="${name}_end1_link"/>
-            <child link="${name}_end2_link"/>
+            <parent link="${name}_pan_link"/>
+            <child link="${name}_tilt_link"/>
             <origin xyz="0.05 -0.015 0.018" rpy="1.57 0 0"/>
             <axis xyz="0 1 0"/>
@@ -60,5 +67,5 @@
         <link name="${name}_end_effector_link"/>
         <joint name="${name}_joint_6" type="fixed">
-            <parent link="${name}_end2_link"/>
+            <parent link="${name}_tilt_link"/>
             <child link="${name}_end_effector_link"/>
             <origin xyz="0.04 -0.016 0" rpy="0 0 0"/>

File: urdf/arm_1.xacro (robot description, xacro)
@@ -6,4 +6,4 @@
     <link name="base_link"/>
     <!-- Arm1 -->
-    <xacro:thorvald_arm name="arm_1" parent="base_link" xyz="0.05 0.55 1.2" rpy="0 0 3.14"/>
+    <xacro:thorvald_arm name="arm1" parent="base_link" xyz="0.05 0.55 1.2" rpy="0 0 3.14"/>
 </robot>

File: urdf/arm_2.xacro (robot description, xacro)
@@ -6,4 +6,4 @@
     <link name="base_link"/>
     <!-- Arm2 -->
-    <xacro:thorvald_arm name="arm_2" parent="base_link" xyz="0.05 -0.55 1.2" rpy="0 0 0"/>
+    <xacro:thorvald_arm name="arm2" parent="base_link" xyz="0.05 -0.55 1.2" rpy="0 0 0"/>
 </robot>

Commit message: test

File: urdf/arm.xacro (robot description, xacro)
@@ -68,8 +68,12 @@
         <joint name="${name}_joint_6" type="fixed">
 <<<<<<< HEAD
+<<<<<<< HEAD
             <parent link="${name}_tilt_link"/>
 =======
             <parent link="${name}_end2_link"/>
 >>>>>>> 0a74866... Add markers to end effector
+=======
+            <parent link="${name}_tilt_link"/>
+>>>>>>> b10cc71... test
             <child link="${name}_end_effector_link"/>
             <origin xyz="0.04 -0.016 0" rpy="0 0 0"/>

Commit message: removed contributer

File: urdf/arm.xacro (robot description, xacro)
@@ -67,13 +67,5 @@
         <link name="${name}_end_effector_link"/>
         <joint name="${name}_joint_6" type="fixed">
-<<<<<<< HEAD
-<<<<<<< HEAD
             <parent link="${name}_tilt_link"/>
-=======
-            <parent link="${name}_end2_link"/>
->>>>>>> 0a74866... Add markers to end effector
-=======
-            <parent link="${name}_tilt_link"/>
->>>>>>> b10cc71... test
             <child link="${name}_end_effector_link"/>
             <origin xyz="0.04 -0.016 0" rpy="0 0 0"/>
